File: Hardware/E90 Kicad Files/E90.sch (KiCad schematic (older format))
At the start: 92 parts, among them J1 Power Connector Conn_01x02, J10 SDIN Jumper, J11 CS_SDOUT Pre Buffer Test Point, J12 SDOUT Jumper, J13 Audio Connector In Conn_01x03, J14 Conn_02x06_Odd_Even, J15 CS Passthru Jumper Conn_01x02, J17 I2S SDIN Bypass Jumper Conn_0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, J18 PMOD Passthru, J19 I2S SDOUT Bypass Conn_01x02, J2 SWD Connector Conn_02x03, J3 Power Test Point Conn_01x02, J4 BOOT0 Test Point, J6 Audio Connector Out Conn_01x03, J7 MCLK Jumper, J8 WS Jumper, J9 SCLK Jumper, U1 AMS1117-3.3, U2 CS4344_CZZ, U3 NC7SZ125P5, U4 CS5343_CZZ, U5 STM32F407VGT60

Commit message: idk
Parts:
- removed C31: 1uF, Capacitor_SMD:C_0603_1608Metric, symbol Device:C_Small
- removed C37: 180pF, Capacitor_SMD:C_0603_1608Metric, symbol Device:C_Small
- removed D3: LED_Red, LED_SMD:LED_0603_1608Metric, symbol Device:LED_Small
- removed D4: LED_Green, LED_SMD:LED_0603_1608Metric, symbol Device:LED_Small
- removed D5: LED_Blue, LED_SMD:LED_0603_1608Metric, symbol Device:LED_Small
- removed D6: LED_Yellow, LED_SMD:LED_0603_1608Metric, symbol Device:LED_Small
- removed J1: Power Connector Conn_01x02, Connector_PinHeader_2.54mm:PinHeader_1x02_P2.54mm_Vertical, symbol Connector_Generic:Conn_01x02
- removed J10: SDIN Jumper, Connector_PinHeader_2.54mm:PinHeader_2x02_P2.54mm_Vertical, symbol Connector_Generic:Conn_02x02_Counter_Clockwise
- removed J11: CS_SDOUT Pre Buffer Test Point, Connector_PinHeader_2.54mm:PinHeader_1x01_P2.54mm_Vertical, symbol Connector_Generic:Conn_01x01
- removed J12: SDOUT Jumper, Connector_PinHeader_2.54mm:PinHeader_2x02_P2.54mm_Vertical, symbol Connector_Generic:Conn_02x02_Counter_Clockwise
- removed J13: Audio Connector In Conn_01x03, Connector_PinHeader_2.54mm:PinHeader_1x03_P2.54mm_Vertical, symbol Connector_Generic:Conn_01x03
- removed J14: Conn_02x06_Odd_Even, Connector_PinHeader_2.54mm:PinHeader_2x06_P2.54mm_Vertical, symbol Connector_Generic:Conn_02x06_Odd_Even
- removed J15: CS Passthru Jumper Conn_01x02, Connector_PinHeader_2.54mm:PinHeader_1x02_P2.54mm_Vertical, symbol Connector_Generic:Conn_01x02
- removed J17: I2S SDIN Bypass Jumper Conn_01x02, Connector_PinHeader_2.54mm:PinHeader_1x02_P2.54mm_Vertical, symbol Connector_Generic:Conn_01x02
- removed J18: PMOD Passthru, Connector_PinHeader_2.54mm:PinHeader_1x02_P2.54mm_Vertical, symbol Connector_Generic:Conn_01x02
- removed J19: I2S SDOUT Bypass Conn_01x02, Connector_PinHeader_2.54mm:PinHeader_1x02_P2.54mm_Vertical, symbol Connector_Generic:Conn_01x02
- removed J4: BOOT0 Test Point, Connector_PinHeader_2.54mm:PinHeader_1x01_P2.54mm_Vertical, symbol Connector_Generic:Conn_01x01
- removed J7: MCLK Jumper, Connector_PinHeader_2.54mm:PinHeader_2x02_P2.54mm_Vertical, symbol Connector_Generic:Conn_02x02_Counter_Clockwise
- removed J8: WS Jumper, Connector_PinHeader_2.54mm:PinHeader_2x02_P2.54mm_Vertical, symbol Connector_Generic:Conn_02x02_Counter_Clockwise
- removed J9: SCLK Jumper, Connector_PinHeader_2.54mm:PinHeader_2x02_P2.54mm_Vertical, symbol Connector_Generic:Conn_02x02_Counter_Clockwise
- removed U3: NC7SZ125P5, SC-70-5, symbol E90_Embedded_DSP:NC7SZ125P5
- added ADC1_IN1, ADC1_IN2, ADC1_IN3: R_POT_US, Potentiometer_THT:Potentiometer_Bourns_PTV09A-1_Single_Vertical, symbol Device:R_POT_US
- added C31: 10uF, Capacitor_SMD:C_0805_2012Metric, symbol Device:CP1_Small
- added D3: B5819W, Diode_SMD:D_SOD-123, symbol Device:D_Schottky_Small
- added D4, D5, D6: LED_RGBA, LED_SMD:19-237-R6GHBHC-A01-2T, symbol Device:LED_RGBA
- added H1, H2, H3, H4: MountingHole_Pad, MountingHole:MountingHole_4.3mm_M4_Pad_Via, symbol Mechanical:MountingHole_Pad
- added InputGain1: 100k, Potentiometer_THT:Potentiometer_Piher_PT-10-V10_Vertical, symbol Device:R_POT_TRIM_US
- added J1, J4: Conn_01x03, Connector_PinHeader_2.54mm:PinHeader_1x03_P2.54mm_Vertical, symbol Connector_Generic:Conn_01x03
- added J10, J9: SJ-63073E, Connector_Audio:CUI_SJ-63073E, symbol Connector:SJ-63073E
- added J5: Conn_01x02, Connector_PinHeader_2.54mm:PinHeader_1x02_P2.54mm_Vertical, symbol Connector_Generic:Conn_01x02
- added J7: USB_B_Mini, Connector_USB:USB_Mini-B_Lumberg_2486_01_Horizontal, symbol Connector:USB_B_Mini
- added J8: Barrel_Jack_Switch, Connector_BarrelJack:BarrelJack_Horizontal, symbol Connector:Barrel_Jack_Switch
- added R21, R31, R32, R33, R34: 10k, Resistor_SMD:R_0603_1608Metric, symbol Device:R_Small_US
- added R22, R23, R24, R25, R26, R27, R28, R29, R30: 1k, Resistor_SMD:R_0603_1608Metric, symbol Device:R_Small_US
- added U3: TLV2774, Package_DIP:DIP-14_W7.62mm_LongPads, symbol E90_Embedded_DSP:TLV2774
- added U6: USBLC6-2SC6, Package_TO_SOT_SMD:SOT-23-6, symbol Power_Protection:USBLC6-2SC6
- added Volume1: 10k, Potentiometer_THT:Potentiometer_Bourns_PTV09A-1_Single_Vertical, symbol Device:R_POT_US
- C11: value 2.7nF -> 10uF; LCSC C1609 -> C19702; LCSC Part # C1609 -> C19702; LCSC part number C1609 -> C19702
- C26: value 100nf -> 10uF; footprint Capacitor_SMD:C_0402_1005Metric -> Capacitor_SMD:C_0603_1608Metric; LCSC C1525 -> C19702; LCSC Part # C1525 -> C19702; LCSC part number C1525 -> C19702
- C6: value 3.3uF -> 10uF; LCSC C51412 -> C19702; LCSC Part # C51412 -> C19702; LCSC part number C51412 -> C19702
- J6: value Audio Connector Out Conn_01x03 -> Conn_01x03
- R12, R9: value 5.1K -> 10k; LCSC C23186 -> C25804; LCSC Part # C23186 -> C25804; LCSC part number C23186 -> C25804
- R15, R16, R17, R18: value 2k2 -> 10k; LCSC C4190 -> C25804; LCSC Part # C4190 -> C23186; LCSC part number C4190 -> C23186
- R19, R20: LCSC Part # C25804 -> C23186; LCSC part number C25804 -> C23186
- R3: value 470 -> 10k; LCSC C23179 -> C25804; LCSC Part # C23179 -> C25804; LCSC part number C23179 -> C25804
- R5: value 10K -> 10k
- U5: LCSC C12345 -> C919362
Connections:
- net labels added: +1.65V, +5V, ADC1_IN1, ADC1_IN2, ADC1_IN3, ANALOG_IN, ANALOG_OUT, CS4344_OUT, CS5343_IN, PA0_PWM, PA6_PWM, PA7_PWM, PB0_PWM, PB11_PWM, PB1_PWM, PD12_PWM, PD13_PWM, PD14_PWM, USB_CONN_D+, USB_CONN_D-, USB_D+, USB_D-
- net labels removed: CS_CLK, CS_MCLK, CS_SDIN, CS_SDOUT, CS_WS, PMOD_CLK, PMOD_MCLK, PMOD_SDIN, PMOD_SDOUT, PMOD_WS
- wire segments 350 -> 379
- no-connect marks 72 -> 64
Other:
- note added: "A/D\n"
- note added: "Attenuator Pot\n"
- note added: "Boot mode selection\n"
- note added: "Center Negative Plug"
- note added: "GPIO"
- note added: "I2C"
- note added: "Input Gain Stage"
- note added: "Output Voltage Follower\n"
- note added: "Parameter Pots\n"
- note added: "Quad OP Amp Circuit IN/OUT"
- note added: "RGB LEDs\n"
- note added: "U3A Unused"
- note added: "U3C Unused\n"
- note added: "assumes CW 2->3\n\n"
- note removed: "A/D"
- note removed: "Configure to Boot from Main Flash\n"
- note removed: "Passthru switch connectors\n"
- note removed: "Switch between onboard (CS) A/D, D/A or external PMOD unit\nJumper Vertical = CS \nJumper horizontal = PMOD"
- moved on the sheet: C1, C10, C12, C13, C14, C15, C16, C17, C18, C19, C2, C20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
